File: car.kicad_pcb (KiCad board)
At the start: 4 copper layers, 116.5 x 104.5 mm, 27 parts, among them J1 Barrel_Jack_MountingPin, J2 L- L+ R- R+, J3 HCSR04, J4 HC05, U1 LM7805 TO220 Horizontal, U2 L293D, U3 NE555P, U4 74HC00

Commit message: rev2
Parts:
- removed C4, C6: 100nF, Capacitor_THT:C_Disc_D3.0mm_W1.6mm_P2.50mm
- removed LED: Conn_01x04_Socket, Connector_PinSocket_2.54mm:PinSocket_1x04_P2.54mm_Vertical
- removed SRV: Servo, Connector_PinHeader_2.54mm:PinHeader_1x03_P2.54mm_Vertical
- added BT1: Battery_Cell, Battery:BatteryHolder_Keystone_1042_1x18650, F.Cu at (76.0, 26.0)
- added BT2: Battery_Cell, Battery:BatteryHolder_Keystone_1042_1x18650, F.Cu at (76.0, 48.5)
- added C10: 100nF, Capacitor_THT:C_Disc_D3.0mm_W1.6mm_P2.50mm, F.Cu at (65.4, 66.0)
- added C12: 100nF, Capacitor_THT:C_Disc_D3.0mm_W1.6mm_P2.50mm, F.Cu at (28.4, 99.5)
- added C13: 100uF, Capacitor_THT:CP_Radial_D5.0mm_P2.00mm, F.Cu at (27.2, 52.0)
- added C7: 100nF, Capacitor_THT:C_Disc_D3.0mm_W1.6mm_P2.50mm, F.Cu at (101.4, 96.5)
- added C8: 100nF, Capacitor_THT:C_Disc_D3.0mm_W1.6mm_P2.50mm, F.Cu at (22.9, 46.5)
- added C9: 100nF, Capacitor_THT:C_Disc_D3.0mm_W1.6mm_P2.50mm, F.Cu at (121.4, 78.5)
- added LED1: REVERSE BRAKE LEFT RIGHT, Connector_PinSocket_2.54mm:PinSocket_1x04_P2.54mm_Vertical, F.Cu at (131.6, 63.9)
- added SRV1: Servo GND +5V PWM, Connector_PinHeader_2.54mm:PinHeader_1x03_P2.54mm_Vertical, F.Cu at (15.1, 69.5)
- added SW1: ON OFF, Button_Switch_THT:SW_Slide_SPDT_Straight_CK_OS102011MS2Q, F.Cu at (28.7, 18.0)
- A1: value Arduino Nano -> Arduino Nano v3; footprint Module:Arduino_Nano -> Arduino:Arduino_Nano
- BZ1: value Horn -> Buzzer
- BZ2: value Alarm -> Buzzer
- C2: value 100uF -> 1uF
- J1: value Barrel_Jack_MountingPin -> GND GND; footprint Connector_BarrelJack:BarrelJack_Horizontal -> Connector_PinHeader_2.54mm:PinHeader_1x02_P2.54mm_Vertical
- J2: value L- L+ R- R+ -> L-L+R-R+
- J3: value HCSR04 -> HCSR04 VCC TRIG ECHO GND
- J4: value HC05 -> HC05 STATE RXD TXD GND VCC EN
- R3: value 1K -> 8K2
- R4: value 3K3 -> 220K
- moved U1 211.9 mm to (19.1, 43.7)
- moved C5 211.6 mm to (17.9, 46.5)
- moved U2 192.5 mm to (27.7, 111.1), turned to 90 degrees
- moved J2 187.6 mm to (68.1, 110.5), turned to 0 degrees
- moved BZ2 159.8 mm to (27.5, 88.0)
- moved C3 157.8 mm to (50.1, 105.5)
- moved BZ1 152.5 mm to (27.5, 71.0)
- moved J3 129.4 mm to (15.1, 51.0)
- moved R5 123.0 mm to (114.8, 62.0)
- moved R6 123.0 mm to (114.8, 66.0)
- moved R7 123.0 mm to (114.8, 70.1)
- moved R8 123.0 mm to (114.8, 74.2)
- moved J4 118.4 mm to (45.1, 70.4), turned to 0 degrees
- moved R2 108.7 mm to (49.9, 66.5), turned to 0 degrees
- moved R1 107.6 mm to (49.6, 73.0)
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Connections:
- net Net-(A1-D9) renamed /SPEED_GPIO_PWM
- net Net-(J2-Pin_1) renamed /R+_OUT
- net Net-(J2-Pin_2) renamed /R-_OUT
- net Net-(J2-Pin_3) renamed /L+_OUT
- net Net-(J2-Pin_4) renamed /L-_OUT
- net Net-(J4-Pin_2) renamed /TX
- net Net-(U3-Q) renamed /555_OUT
- A1 pad 10: Net-(A1-D7) -> /L+_GPIO
- A1 pad 11: Net-(A1-D8) -> /L-_GPIO
- A1 pad 13: Net-(A1-D10) -> /HORN_GPIO_PWM
- A1 pad 14: Net-(A1-D11) -> /ALARM_GPIO_PWM
- A1 pad 15: Net-(A1-D12) -> /REVERSE_GPIO
- A1 pad 16: Net-(A1-D13) -> /BRAKE_GPIO
- A1 pad 19: Net-(A1-A0) -> /TLEFT_GPIO
- A1 pad 20: Net-(A1-A1) -> /TRIGHT_GPIO
- A1 pad 21: Net-(A1-A2) -> /RX_GPIO
- A1 pad 22: Net-(A1-A3) -> /TX_GPIO
- A1 pad 5: /REVERSE_GPIO -> /TRIG_GPIO
- A1 pad 6: /ALARM -> /SERVO_GPIO_PWM
- A1 pad 7: /BRAKE_GPIO -> /ECHO_GPIO
- A1 pad 8: /TLEFT_GPIO -> /R+_GPIO
- A1 pad 9: /TRIGHT_GPIO -> /R-_GPIO
- BZ1 pad 1: Net-(A1-D11) -> /HORN_GPIO_PWM
- BZ2 pad 1: /ALARM -> /ALARM_GPIO_PWM
- C1 pad 1: Net-(U3-CV) -> GND
- C1 pad 2: GND -> Net-(U3-CV)
- C3 pad 1: Net-(U1-VI) -> +BATT
- C5 pad 1: +5V -> +BATT
- J1 pad 1: Net-(U1-VI) -> GND
- J3 pad 2: Net-(A1-D8) -> /ECHO_GPIO
- J3 pad 3: Net-(A1-D7) -> /TRIG_GPIO
- J4 pad 3: Net-(A1-D13) -> /RX_GPIO
- R2 pad 2: Net-(A1-D12) -> /TX_GPIO
- U1 pad 1: Net-(U1-VI) -> +BATT
- U2 pad 10: Net-(A1-A2) -> /L+_GPIO
- U2 pad 15: Net-(A1-A3) -> /L-_GPIO
- U2 pad 2: Net-(A1-A0) -> /R+_GPIO
- U2 pad 7: Net-(A1-A1) -> /R-_GPIO
- U2 pad 8: Net-(U1-VI) -> +BATT
- U4 pad 1: GND -> Net-(U4-Pad1)
- U4 pad 11: Net-(R8-Pad1) -> Net-(U4-Pad11)
- U4 pad 2: GND -> Net-(U4-Pad1)
- U4 pad 3: unconnected-(U4-Pad3) -> Net-(R7-Pad1)
- U4 pad 4: GND -> Net-(U4-Pad11)
- U4 pad 5: GND -> Net-(U4-Pad11)
- U4 pad 6: unconnected-(U4-Pad6) -> Net-(R8-Pad1)
- U4 pad 8: Net-(R7-Pad1) -> Net-(U4-Pad1)
Routing:
- net +BATT: track 0.00 -> 134.4 mm
- net /TRIG_GPIO: track 0.00 -> 103.7 mm
- net Net-(BT1--): track 0.00 -> 96.7 mm
- net Net-(A1-D11): track 91.8 -> 0.00 mm
- net /ECHO_GPIO: track 0.00 -> 89.7 mm
- net /R-_GPIO: track 0.00 -> 77.2 mm
- net /L+_GPIO: track 0.00 -> 76.1 mm
- net /HORN_GPIO_PWM: track 0.00 -> 76.1 mm
- net /SERVO_GPIO_PWM: track 0.00 -> 75.5 mm
- net Net-(U1-VI): track 72.8 -> 0.00 mm
- net /ALARM_GPIO_PWM: track 0.00 -> 67.9 mm
- net Net-(A1-A0): track 63.7 -> 0.00 mm
- net /L-_GPIO: track 0.00 -> 61.3 mm
- net Net-(A1-A3): track 60.8 -> 0.00 mm
- net /REVERSE_GPIO: track 89.8 -> 31.7 mm
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- added copper zone on In2.Cu, net GND
- removed copper zone on B.Cu, net GND
Other:
- board size 116.5 x 104.5 mm -> 124 x 104 mm
- board text removed: "GND ECHO TRIG VCC"
- board text removed: "GND VCC PWM"
- board text removed: "REV BRK L R"
- board text removed: "STATE RXD TXD GND VCC EN"
